File: BatteryPCB/BatteryPCB.kicad_sch (KiCad schematic)
At the start: 18 parts, among them J1 Conn_01x01, J2 Conn_01x01, J3 Conn_01x01, J4 Conn_01x01_Socket, SW1 SW_SPST, SW2 SW_SPST, U1 L7805CV, U2 R24-150B, U3 R24-150B

Commit message: Updates from 3/29 comments
Parts:
- removed SW1, SW2: SW_SPST, Button_Switch_THT:SW_DIP_SPSTx02_Slide_6.7x6.64mm_W7.62mm_P2.54mm_LowProfile, symbol Switch:SW_SPST
- removed U2, U3: R24-150B, RXX-100_150B_RCP, symbol R24-150B:R24-150B
- added SW1, SW3: ANT11TFHQE, 100SP1T1B4M2QE:100SP1T1_EWI, symbol Switch:SW_DPDT_x2
- added U2, U3: R05-100B, Package_DIP:DIP-24_W15.24mm, symbol R05_100B:R05-100B
- U1: value L7805CV -> LF50CV
Connections:
- net +5V: now also C3.2, C5.2, SW1.2 (B), U2.22 (+VIN), U2.23 (+VIN), U3.22 (+VIN), U3.23 (+VIN)
- net -VSW: now also U3.15 (-VOUT); no longer BT1.2 (-), C1.2, C2.2, C4.2, C6.2, J3.1 (Pin_1), RV1.3, RV2.3, U1.2 (GROUND)
- net HT: now also U2.12 (+VOUT), U2.13 (+VOUT)
- net at RV2.1: now also U3.16 (VREF), U3.9 (VREF)
- net at RV2.2: now also U3.17 (VADJ), U3.8 (VADJJ)
- net at C6.1: now also U3.12 (+VOUT), U3.13 (+VOUT)
- net GND: now reaches C3.1, C5.1
- net GND: now also BT1.2 (-), C1.2, C2.2, C4.2, C6.2, J3.1 (Pin_1), RV1.3, RV2.3, U1.2 (GROUND), SW1.3 (C), U2.10 (-VOUT), U2.15 (-VOUT), U2.2 (-VIN), U2.3 (-VIN), U3.10 (-VOUT), U3.2 (-VIN), U3.3 (-VIN)
- net at C2.1, U1.1 (INPUT): now also SW3.3 (C)
- net at RV1.1: now also U2.16 (VREF), U2.9 (VREF)
- net at RV1.2: now also U2.17 (VADJ), U2.8 (VADJJ)
- net at BT1.1 (+): now also SW3.2 (B)

Commit message: In progress changes from 3/29 2nd comments
Parts:
- removed SW1, SW3: ANT11TFHQE, 100SP1T1B4M2QE:100SP1T1_EWI, symbol Switch:SW_DPDT_x2
- removed U1: LF50CV, L7805CV:TO-220_STM, symbol L7805CV:L7805CV
- removed U2, U3: R05-100B, Package_DIP:DIP-24_W15.24mm, symbol R05_100B:R05-100B
- added SW1, SW2: ANT11TFHQE, 100SP1T1B4M2QE:100SP1T1_EWI, symbol Switch:SW_DIP_x01
- added U1: LF50CV, TO-220_STM, symbol LF50CV:LF50CV
- added U2, U3: R05-100B, Package_DIP:DIP-24_W15.24mm, symbol InTENS_customparts:R05-100B
- RV1, RV2: value 5kΩ -> R_Potentiometer_US; footprint Potentiometer_THT:Potentiometer_ACP_CA6-H2,5_Horizontal -> (none)
- renumbered C2 to C1, C1 to C2
Connections:
- net -VSW: now also C6.1, RV1.3, U3.10 (-VOUT), U3.15 (-VOUT)
- net GND: now also C4.1, U1.2 (GND), U2.10 (-VOUT), U2.15 (-VOUT), U2.2 (-VIN), U2.3 (-VIN), U3.12 (+VOUT), U3.13 (+VOUT), U3.2 (-VIN), U3.3 (-VIN); no longer C4.2, RV1.3
- net HT: now also C4.2, U2.12 (+VOUT), U2.13 (+VOUT); no longer C4.1
- net at RV2.1: now also U2.16 (VREF), U2.9 (VREF)
- net at RV2.2: now also U2.17 (VADJ), U2.8 (VADJ)
- net at RV1.1: now also U3.16 (VREF), U3.9 (VREF)
- net at RV1.2: now also U3.17 (VADJ), U3.8 (VADJ)
- net at BT1.1 (+): now also SW1.1
- net at C1.1: now also SW1.2, U1.1 (IN)
- net +5V: no longer names the net of C3.2, C5.2
- net +5V: now also SW2.2, U2.22 (+VIN), U2.23 (+VIN), U3.22 (+VIN), U3.23 (+VIN); no longer C2.1
- new net: C2.1, SW2.1, U1.3 (OUT)
Other:
- moved on the sheet: BT1, C1, C2, C3, C4, C5, C6, J1, J2, J3, J4

Commit message: 2nd Update from 3/29 comments
Parts:
- J4: footprint Connector_Wuerth:Wuerth_WR-WTB_64800211622_1x02_P1.50mm_Vertical -> Connector_PinSocket_2.54mm:PinSocket_1x02_P2.54mm_Vertical
- RV1, RV2: value R_Potentiometer_US -> 93PR5KLF; footprint (none) -> 93PR5KL:RES3_93_TTE
- U1: footprint TO-220_STM -> LF50CV:LF50CV
Connections:
- net +5V: now reaches C2.1, SW2.1, U1.3 (OUT)
Other:
- moved on the sheet: BT1, C1, C2, SW1, U1

Commit message: Updated from 3/30 comments
Parts:
- RV1, RV2: value 93PR5KLF -> CT-6EP502; footprint 93PR5KL:RES3_93_TTE -> Potentiometer_THT:Potentiometer_Bourns_3006P_Horizontal
Changed lines of the file:
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@@
+	)
+	(symbol
+		(lib_id "Device:R_Potentiometer_US")
+		(at 215.9 68.58 90)
+		(unit 1)
+		(exclude_from_sim no)
+		(in_bom yes)
+		(on_board yes)
+		(dnp no)
+		(fields_autoplaced yes)
+		(property "Reference" "RV2"
+			(at 215.9 72.39 90)
+			(effects
+				(font
+					(size 1.27 1.27)
+				)
+			)
+		)
+		(property "Value" "CT-6EP502"
+			(at 215.9 74.93 90)
+			(effects
+				(font
+					(size 1.27 1.27)
+				)
+			)
+		)
+		(property "Footprint" "Potentiometer_THT:Potentiometer_Bourns_3006P_Horizontal"
+			(at 215.9 68.58 0)
+			(effects
+				(font
+					(size 1.27 1.27)
+				)
+				(hide yes)
+			)
+		)
+		(property "Datasheet" "~"
+			(at 215.9 68.58 0)
+			(effects
+				(font
+					(size 1.27 1.27)
+				)
+				(hide yes)
+			)
+		)
+		(property "Description" ""
+			(at 215.9 68.58 0)
+			(effects
+				(font
+					(size 1.27 1.27)
+				)
+				(hide yes)
+			)
+		)
+		(pin "2"
+		)
+		(pin "3"
+		)
+		(pin "1"
+		)
+		(instances
+			(project "BatteryPCB"
+				(path "/e63e39d7-6ac0-4ffd-8aa3-1841a4541b55"
+					(reference "RV2")
+					(unit 1)
+				)
+			)
+		)
 	)
 	(symbol
@@
 	)
 	(symbol
-		(lib_id "Device:R_Potentiometer_US")
-		(at 215.9 68.58 90)
-		(unit 1)
-		(exclude_from_sim no)
-		(in_bom yes)
-		(on_board yes)
-		(dnp no)
-		(fields_autoplaced yes)
-		(property "Reference" "RV2"
-			(at 215.9 72.39 90)
-			(effects
-				(font
-					(size 1.27 1.27)
-				)
-			)
-		)
-		(property "Value" "93PR5KLF"
-			(at 215.9 74.93 90)
-			(effects
-				(font
-					(size 1.27 1.27)
-				)
-			)
-		)
-		(property "Footprint" "93PR5KL:RES3_93_TTE"
-			(at 215.9 68.58 0)
-			(effects
-				(font
-					(size 1.27 1.27)
-				)
-				(hide yes)
-			)
-		)
-		(property "Datasheet" "~"
-			(at 215.9 68.58 0)
-			(effects
-				(font
-					(size 1.27 1.27)
-				)
-				(hide yes)
-			)
-		)
-		(property "Description" ""
-			(at 215.9 68.58 0)
-			(effects
-				(font
-					(size 1.27 1.27)
-				)
-				(hide yes)
-			)
-		)
-		(pin "2"
-		)
-		(pin "3"
-		)
-		(pin "1"
-		)
-		(instances
-			(project "BatteryPCB"
-				(path "/e63e39d7-6ac0-4ffd-8aa3-1841a4541b55"
-					(reference "RV2")
-					(unit 1)
-				)
-			)
-		)
-	)
-	(symbol
 		(lib_id "Device:C")
 		(at 72.39 50.8 0)
@@
 			)
 		)
-		(property "Value" "93PR5KLF"
+		(property "Value" "CT-6EP502"
 			(at 215.9 143.51 90)
 			(effects
@@
 			)
 		)
-		(property "Footprint" "93PR5KL:RES3_93_TTE"
+		(property "Footprint" "Potentiometer_THT:Potentiometer_Bourns_3006P_Horizontal"
 			(at 215.9 137.16 0)
 			(effects

Commit message: Updated from 3/30 comments
Parts:
- RV1, RV2: value CT-6EP502 -> 3006P-1-502LF
Changed lines of the file:
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@@
 			)
 		)
-		(property "Value" "CT-6EP502"
+		(property "Value" "3006P-1-502LF"
 			(at 215.9 74.93 90)
 			(effects
@@
 			)
 		)
-		(property "Value" "CT-6EP502"
+		(property "Value" "3006P-1-502LF"
 			(at 215.9 143.51 90)
 			(effects

Commit message: 4/1 trim pot change
Parts:
- RV1, RV2: value 3006P-1-502LF -> 64WR5KLF; footprint Potentiometer_THT:Potentiometer_Bourns_3006P_Horizontal -> 64WR5KLF:RES3_64W_TTE
Changed lines of the file:
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@@
 			)
 		)
-		(property "Value" "3006P-1-502LF"
+		(property "Value" "64WR5KLF"
 			(at 215.9 74.93 90)
 			(effects
@@
 			)
 		)
-		(property "Footprint" "Potentiometer_THT:Potentiometer_Bourns_3006P_Horizontal"
+		(property "Footprint" "64WR5KLF:RES3_64W_TTE"
 			(at 215.9 68.58 0)
 			(effects
@@
 			)
 		)
-		(property "Value" "3006P-1-502LF"
+		(property "Value" "64WR5KLF"
 			(at 215.9 143.51 90)
 			(effects
@@
 			)
 		)
-		(property "Footprint" "Potentiometer_THT:Potentiometer_Bourns_3006P_Horizontal"
+		(property "Footprint" "64WR5KLF:RES3_64W_TTE"
 			(at 215.9 137.16 0)
 			(effects
